File: Radioberry-I-O.kicad_pcb (KiCad board)
At the start: 2 copper layers, 85 x 56 mm, 36 parts, among them CN1 RCA Jack, CN2 RCA Jack, CN3 3.5mm stereo jack, CN4 3.5mm stereo jack, CN5 3.5mm stereo jack, J1 2x10 female header 2.54mm, J2 2x7 male header 2.54mm, M1 30mm Fan, Q1 NUD3124LT1G, Q2 NUD3124LT1G

Commit message: BOM cleanup
Parts:
- Q1, Q2: value NUD3124LT1G -> NUD3160LT1G
Changed lines of the file:
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@@
     (descr "Resistor SMD 0603 (1608 Metric), square (rectangular) end terminal, IPC_7351 nominal, (Body size source: IPC-SM-782 page 72, https://www.pcb-3d.com/wordpress/wp-content/uploads/ipc-sm-782a_amendment_1_and_2.pdf), generated with kicad-footprint-generator")
     (tags "resistor")
-    (property "Part Number" "CR0603-10W-000T")
+    (property "Part Number" "RC0603JR-130RL")
     (property "Sheetfile" "Radioberry-I-O.kicad_sch")
     (property "Sheetname" "")
@@
     (descr "Resistor SMD 0603 (1608 Metric), square (rectangular) end terminal, IPC_7351 nominal, (Body size source: IPC-SM-782 page 72, https://www.pcb-3d.com/wordpress/wp-content/uploads/ipc-sm-782a_amendment_1_and_2.pdf), generated with kicad-footprint-generator")
     (tags "resistor")
-    (property "Part Number" "CR0603-10W-000T")
+    (property "Part Number" "RC0603JR-130RL")
     (property "Sheetfile" "Radioberry-I-O.kicad_sch")
     (property "Sheetname" "")
@@
     (descr "Resistor SMD 0603 (1608 Metric), square (rectangular) end terminal, IPC_7351 nominal, (Body size source: IPC-SM-782 page 72, https://www.pcb-3d.com/wordpress/wp-content/uploads/ipc-sm-782a_amendment_1_and_2.pdf), generated with kicad-footprint-generator")
     (tags "resistor")
-    (property "Part Number" "CR0603-10W-000T")
+    (property "Part Number" "RC0603JR-130RL")
     (property "Sheetfile" "Radioberry-I-O.kicad_sch")
     (property "Sheetname" "")
@@
   (footprint "Radioberry-I-O:SOT23_3" (layer "B.Cu")
     (at 63.9 66.4 180)
-    (property "Part Number" "NUD3124LT1G")
+    (property "Part Number" "NUD3160LT1G")
     (property "Sheetfile" "Radioberry-I-O.kicad_sch")
     (property "Sheetname" "")
@@
       (effects (font (size 0.8 0.8) (thickness 0.1)) (justify mirror))
     )
-    (fp_text value "NUD3124LT1G" (at 0 3.4) (layer "B.Fab") hide
+    (fp_text value "NUD3160LT1G" (at 0 3.4) (layer "B.Fab") hide
       (effects (font (size 0.8 0.8) (thickness 0.1)) (justify mirror))
     )
@@
     (descr "Resistor SMD 0603 (1608 Metric), square (rectangular) end terminal, IPC_7351 nominal, (Body size source: IPC-SM-782 page 72, https://www.pcb-3d.com/wordpress/wp-content/uploads/ipc-sm-782a_amendment_1_and_2.pdf), generated with kicad-footprint-generator")
     (tags "resistor")
-    (property "Part Number" "CR0603-10W-000T")
+    (property "Part Number" "RC0603JR-130RL")
     (property "Sheetfile" "Radioberry-I-O.kicad_sch")
     (property "Sheetname" "")
@@
     (descr "Resistor SMD 0603 (1608 Metric), square (rectangular) end terminal, IPC_7351 nominal, (Body size source: IPC-SM-782 page 72, https://www.pcb-3d.com/wordpress/wp-content/uploads/ipc-sm-782a_amendment_1_and_2.pdf), generated with kicad-footprint-generator")
     (tags "resistor")
-    (property "Part Number" "CR0603-10W-000T")
+    (property "Part Number" "RC0603JR-130RL")
     (property "Sheetfile" "Radioberry-I-O.kicad_sch")
     (property "Sheetname" "")
@@
   (footprint "Radioberry-I-O:SOT23_3" (layer "B.Cu")
     (at 63.7 84.5 180)
-    (property "Part Number" "NUD3124LT1G")
+    (property "Part Number" "NUD3160LT1G")
     (property "Sheetfile" "Radioberry-I-O.kicad_sch")
     (property "Sheetname" "")
@@
       (effects (font (size 0.8 0.8) (thickness 0.1)) (justify mirror))
     )
-    (fp_text value "NUD3124LT1G" (at 0 3.4) (layer "B.Fab") hide
+    (fp_text value "NUD3160LT1G" (at 0 3.4) (layer "B.Fab") hide
       (effects (font (size 0.8 0.8) (thickness 0.1)) (justify mirror))
     )
@@
     (descr "Resistor SMD 0603 (1608 Metric), square (rectangular) end terminal, IPC_7351 nominal, (Body size source: IPC-SM-782 page 72, https://www.pcb-3d.com/wordpress/wp-content/uploads/ipc-sm-782a_amendment_1_and_2.pdf), generated with kicad-footprint-generator")
     (tags "resistor")
-    (property "Part Number" "CR0603-10W-000T")
+    (property "Part Number" "RC0603JR-130RL")
     (property "Sheetfile" "Radioberry-I-O.kicad_sch")
     (property "Sheetname" "")
@@
     (descr "Resistor SMD 0603 (1608 Metric), square (rectangular) end terminal, IPC_7351 nominal, (Body size source: IPC-SM-782 page 72, https://www.pcb-3d.com/wordpress/wp-content/uploads/ipc-sm-782a_amendment_1_and_2.pdf), generated with kicad-footprint-generator")
     (tags "resistor")
-    (property "Part Number" "CR0603-10W-000T")
+    (property "Part Number" "RC0603JR-130RL")
     (property "Sheetfile" "Radioberry-I-O.kicad_sch")
     (property "Sheetname" "")
@@
     (descr "Resistor SMD 0603 (1608 Metric), square (rectangular) end terminal, IPC_7351 nominal, (Body size source: IPC-SM-782 page 72, https://www.pcb-3d.com/wordpress/wp-content/uploads/ipc-sm-782a_amendment_1_and_2.pdf), generated with kicad-footprint-generator")
     (tags "resistor")
-    (property "Part Number" "CR0603-10W-000T")
-    (property "Sheetfile" "Radioberry-I-O.kicad_sch")
-    (property "Sheetname" "")
+    (property "Part Number" "RC0603JR-130RL")
+    (property "Sheetfile" "Radioberry-I-O.kicad_sch")
+    (property "Sheetname" "")
