File: Radioberry-I-O.kicad_sch (KiCad schematic)
At the start: 32 parts, among them CN1 RCA Jack, CN2 RCA Jack, CN3 3.5mm stereo jack, CN4 3.5mm stereo jack, CN5 3.5mm stereo jack, J1 2x10 female header 2.54mm, J2 2x7 male header 2.54mm, M1 30mm Fan, Q1 NUD3124LT1G, Q2 NUD3124LT1G

Commit message: BOM cleanup
Parts:
- Q1, Q2: value NUD3124LT1G -> NUD3160LT1G; Part Number NUD3124LT1G -> NUD3160LT1G
- R101, R102, R103, R104, R105, R106, R107, R108: Part Number CR0603-10W-000T -> RC0603JR-130RL
Changed lines of the file:
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@@
       (effects (font (size 1.27 1.27)) hide)
     )
-    (property "Datasheet" "https://page.venkel.com/hubfs/Resources/Datasheets/CR-Series.pdf" (id 3) (at 32.385 96.52 0)
-      (effects (font (size 1.27 1.27)) hide)
-    )
-    (property "Part Number" "CR0603-10W-000T" (id 4) (at 32.385 96.52 0)
+    (property "Datasheet" "https://www.yageo.com/upload/media/product/productsearch/datasheet/rchip/PYu-RC_Group_51_RoHS_L_11.pdf" (id 3) (at 32.385 96.52 0)
+      (effects (font (size 1.27 1.27)) hide)
+    )
+    (property "Part Number" "RC0603JR-130RL" (id 4) (at 32.385 96.52 0)
       (effects (font (size 1.27 1.27)) hide)
     )
@@
       (effects (font (size 1.27 1.27)) hide)
     )
-    (property "Datasheet" "https://page.venkel.com/hubfs/Resources/Datasheets/CR-Series.pdf" (id 3) (at 49.53 96.52 0)
-      (effects (font (size 1.27 1.27)) hide)
-    )
-    (property "Part Number" "CR0603-10W-000T" (id 4) (at 49.53 96.52 0)
+    (property "Datasheet" "https://www.yageo.com/upload/media/product/productsearch/datasheet/rchip/PYu-RC_Group_51_RoHS_L_11.pdf" (id 3) (at 49.53 96.52 0)
+      (effects (font (size 1.27 1.27)) hide)
+    )
+    (property "Part Number" "RC0603JR-130RL" (id 4) (at 49.53 96.52 0)
       (effects (font (size 1.27 1.27)) hide)
     )
@@
       (effects (font (size 0.9906 0.9906)) (justify left))
     )
-    (property "Value" "NUD3124LT1G" (id 1) (at 245.745 43.1799 0)
+    (property "Value" "NUD3160LT1G" (id 1) (at 245.745 43.1799 0)
       (effects (font (size 0.9906 0.9906)) (justify left))
     )
@@
       (effects (font (size 1.524 1.524)) hide)
     )
-    (property "Datasheet" "https://www.onsemi.com/pdf/datasheet/nud3124-d.pdf" (id 3) (at 241.3 41.275 0)
+    (property "Datasheet" "https://www.onsemi.com/pdf/datasheet/nud3160-d.pdf" (id 3) (at 241.3 41.275 0)
       (effects (font (size 1.524 1.524)) hide)
     )
-    (property "Part Number" "NUD3124LT1G" (id 4) (at 241.3 41.275 0)
+    (property "Part Number" "NUD3160LT1G" (id 4) (at 241.3 41.275 0)
       (effects (font (size 1.27 1.27)) hide)
     )
@@
       (effects (font (size 1.27 1.27)) hide)
     )
-    (property "Datasheet" "https://page.venkel.com/hubfs/Resources/Datasheets/CR-Series.pdf" (id 3) (at 112.395 93.98 0)
-      (effects (font (size 1.27 1.27)) hide)
-    )
-    (property "Part Number" "CR0603-10W-000T" (id 4) (at 112.395 93.98 0)
+    (property "Datasheet" "https://www.yageo.com/upload/media/product/productsearch/datasheet/rchip/PYu-RC_Group_51_RoHS_L_11.pdf" (id 3) (at 112.395 93.98 0)
+      (effects (font (size 1.27 1.27)) hide)
+    )
+    (property "Part Number" "RC0603JR-130RL" (id 4) (at 112.395 93.98 0)
       (effects (font (size 1.27 1.27)) hide)
     )
@@
       (effects (font (size 1.27 1.27)) hide)
     )
-    (property "Datasheet" "https://page.venkel.com/hubfs/Resources/Datasheets/CR-Series.pdf" (id 3) (at 167.64 93.345 0)
-      (effects (font (size 1.27 1.27)) hide)
-    )
-    (property "Part Number" "CR0603-10W-000T" (id 4) (at 167.64 93.345 0)
+    (property "Datasheet" "https://www.yageo.com/upload/media/product/productsearch/datasheet/rchip/PYu-RC_Group_51_RoHS_L_11.pdf" (id 3) (at 167.64 93.345 0)
+      (effects (font (size 1.27 1.27)) hide)
+    )
+    (property "Part Number" "RC0603JR-130RL" (id 4) (at 167.64 93.345 0)
       (effects (font (size 1.27 1.27)) hide)
     )
@@
       (effects (font (size 1.27 1.27)) hide)
     )
-    (property "Datasheet" "https://page.venkel.com/hubfs/Resources/Datasheets/CR-Series.pdf" (id 3) (at 120.65 93.98 0)
-      (effects (font (size 1.27 1.27)) hide)
-    )
-    (property "Part Number" "CR0603-10W-000T" (id 4) (at 120.65 93.98 0)
+    (property "Datasheet" "https://www.yageo.com/upload/media/product/productsearch/datasheet/rchip/PYu-RC_Group_51_RoHS_L_11.pdf" (id 3) (at 120.65 93.98 0)
+      (effects (font (size 1.27 1.27)) hide)
+    )
+    (property "Part Number" "RC0603JR-130RL" (id 4) (at 120.65 93.98 0)
       (effects (font (size 1.27 1.27)) hide)
     )
@@
       (effects (font (size 0.9906 0.9906)) (justify left))
     )
-    (property "Value" "NUD3124LT1G" (id 1) (at 189.865 42.5449 0)
+    (property "Value" "NUD3160LT1G" (id 1) (at 189.865 42.5449 0)
       (effects (font (size 0.9906 0.9906)) (justify left))
     )
@@
       (effects (font (size 1.524 1.524)) hide)
     )
-    (property "Datasheet" "https://www.onsemi.com/pdf/datasheet/nud3124-d.pdf" (id 3) (at 186.055 40.64 0)
+    (property "Datasheet" "https://www.onsemi.com/pdf/datasheet/nud3160-d.pdf" (id 3) (at 186.055 40.64 0)
       (effects (font (size 1.524 1.524)) hide)
     )
-    (property "Part Number" "NUD3124LT1G" (id 4) (at 186.055 40.64 0)
+    (property "Part Number" "NUD3160LT1G" (id 4) (at 186.055 40.64 0)
       (effects (font (size 1.27 1.27)) hide)
     )
@@
       (effects (font (size 1.27 1.27)) hide)
     )
-    (property "Datasheet" "https://page.venkel.com/hubfs/Resources/Datasheets/CR-Series.pdf" (id 3) (at 40.64 96.52 0)
-      (effects (font (size 1.27 1.27)) hide)
-    )
-    (property "Part Number" "CR0603-10W-000T" (id 4) (at 40.64 96.52 0)
+    (property "Datasheet" "https://www.yageo.com/upload/media/product/productsearch/datasheet/rchip/PYu-RC_Group_51_RoHS_L_11.pdf" (id 3) (at 40.64 96.52 0)
+      (effects (font (size 1.27 1.27)) hide)
+    )
+    (property "Part Number" "RC0603JR-130RL" (id 4) (at 40.64 96.52 0)
       (effects (font (size 1.27 1.27)) hide)
     )
@@
       (effects (font (size 1.27 1.27)) hide)
     )
-    (property "Datasheet" "https://page.venkel.com/hubfs/Resources/Datasheets/CR-Series.pdf" (id 3) (at 57.785 96.52 0)
-      (effects (font (size 1.27 1.27)) hide)
-    )
-    (property "Part Number" "CR0603-10W-000T" (id 4) (at 57.785 96.52 0)
+    (property "Datasheet" "https://www.yageo.com/upload/media/product/productsearch/datasheet/rchip/PYu-RC_Group_51_RoHS_L_11.pdf" (id 3) (at 57.785 96.52 0)
+      (effects (font (size 1.27 1.27)) hide)
+    )
+    (property "Part Number" "RC0603JR-130RL" (id 4) (at 57.785 96.52 0)
       (effects (font (size 1.27 1.27)) hide)
     )
@@
       (effects (font (size 1.27 1.27)) hide)
     )
-    (property "Datasheet" "https://page.venkel.com/hubfs/Resources/Datasheets/CR-Series.pdf" (id 3) (at 159.385 93.345 0)
-      (effects (font (size 1.27 1.27)) hide)
-    )
-    (property "Part Number" "CR0603-10W-000T" (id 4) (at 159.385 93.345 0)
+    (property "Datasheet" "https://www.yageo.com/upload/media/product/productsearch/datasheet/rchip/PYu-RC_Group_51_RoHS_L_11.pdf" (id 3) (at 159.385 93.345 0)
+      (effects (font (size 1.27 1.27)) hide)
+    )
+    (property "Part Number" "RC0603JR-130RL" (id 4) (at 159.385 93.345 0)
       (effects (font (size 1.27 1.27)) hide)
     )
@@
     )
     (path "/3fb1b5fd-17ff-457e-aac9-f43a3f9efce7"
-      (reference "Q1") (unit 1) (value "NUD3124LT1G") (footprint "Radioberry-I-O:SOT23_3")
+      (reference "Q1") (unit 1) (value "NUD3160LT1G") (footprint "Radioberry-I-O:SOT23_3")
     )
     (path "/9be540f9-c35f-4a0f-9a89-1391f5f30335"
-      (reference "Q2") (unit 1) (value "NUD3124LT1G") (footprint "Radioberry-I-O:SOT23_3")
+      (reference "Q2") (unit 1) (value "NUD3160LT1G") (footprint "Radioberry-I-O:SOT23_3")
     )
     (path "/014f1669-ae08-450a-b680-baefaf87ddba"

Commit message: Update BOM & readme
Parts:
- M1: Part Number MR3010H05B-RSR -> 3368
Changed lines of the file:
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@@
       (effects (font (size 1.27 1.27)) hide)
     )
-    (property "Datasheet" "https://www.mechatronics.com/pdf/MR3010.pdf" (id 3) (at 131.191 28.575 0)
+    (property "Datasheet" "https://media.digikey.com/pdf/Data%20Sheets/Adafruit%20PDFs/3368_Web.pdf" (id 3) (at 131.191 28.575 0)
       (effects (font (size 1.27 1.27)) hide)
     )
-    (property "Part Number" "MR3010H05B-RSR" (id 4) (at 131.445 28.575 0)
+    (property "Part Number" "3368" (id 4) (at 131.445 28.575 0)
       (effects (font (size 1.27 1.27)) hide)
     )
